File: PCB/PCB.brd (EAGLE design)
At the start: 23 parts, among them IC1 MEGA8-P, Q1 16000

Commit message: diseño final del PCB
Parts:
- moved C3 42.1 mm to (41.9, 55.9)
- moved C4 41.9 mm to (36.8, 55.9)
- moved C2 41.3 mm to (40.6, 83.1), turned to 90 degrees
- moved R1 34.4 mm to (39.4, 63.5)
- moved Q1 28.0 mm to (43.2, 50.8)
- moved D3 20.9 mm to (40.6, 71.3), turned to 270 degrees
- moved RESET 1.45 mm to (97.6, 38.1)
Connections:
- net RXD: now also R4.1; no longer R7.1
- net TXD: now also R7.1; no longer R4.1
Routing:
- net RXD: track 33.9 -> 211.9 mm
- net TXD: track 208.0 -> 33.2 mm
- net N$2: track 68.1 -> 52.6 mm
- net N$24: track 58.0 -> 43.8 mm
- net RES1: track 219.5 -> 227.4 mm
- net N$27: track 74.9 -> 67.6 mm, vias 2 -> 0
- net N$5: track 151.7 -> 147.4 mm
- net GND: track 214.8 -> 210.7 mm
- net +5V: track 257.4 -> 254.7 mm
- net N$4: track 23.8 -> 25.8 mm
- net N$16: track 69.9 -> 69.0 mm, vias 2 -> 0
- net N$1: track 69.1 -> 69.8 mm
Other:
- board text added: "AN1"
- board text added: "AN2"
- board text added: "AN3"
- board text added: "AN4"
- board text added: "AN5"
- board text added: "AN6"
- board text added: "MALUDA 1.0.1"
- board text added: "PINES ANALOGICOS"
- board text added: "PINES DIGITALES"
- board text added: "RESET"
- board text added: "mmmm"
